Commit message: update demo with modif made on fixed version

File: agimus_demo_07_tiago_pro_deburring/urdf/pylone.urdf.xacro (robot description, xacro)
@@ -1,4 +1,4 @@
 <?xml version="1.0" encoding="utf-8"?>
-<robot name="pylone">
+<robot name="pylone" xmlns:xacro="http://www.ros.org/wiki/xacro">
   <material name="grey">
     <color rgba="0.0 0.9 0.9 1.0"/>
@@ -7,5 +7,5 @@
     <visual>
       <geometry>
-        <mesh filename="package://agimus_demo_07_tiago_pro_deburring/urdf/visual/pylone.stl"
+        <mesh filename="file://$(find agimus_demo_07_tiago_pro_deburring)/urdf/visual/pylone.stl"
               scale="1.0 1.0 1.0"/>
       </geometry>
@@ -14,5 +14,5 @@
     <collision>
       <geometry>
-        <mesh filename="package://agimus_demo_07_tiago_pro_deburring/urdf/collision/pylone.stl"
+        <mesh filename="file://$(find agimus_demo_07_tiago_pro_deburring)/urdf/collision/pylone.stl"
               scale="1.0 1.0 1.0"/>
       </geometry>
@@ -24,3 +24,6 @@
     </inertial>
   </link>
+  <gazebo>
+    <static>true</static>
+  </gazebo>
 </robot>
