Commit message: Reduce object size and fix urdf

File: agimus_demo_07_tiago_pro_pick_and_drop/urdf/obj_01.urdf (robot description, URDF)
Before this commit: robot obj_000001, 1 links, 0 joints
Links:
- link base_link: geometry collision mesh filename=package://agimus_demo_07_tiago_pro_pick_and_drop/urdf/obj_0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 scale=1 1 1; visual mesh filename=package://agimus_demo_07_tiago_pro_pick_and_drop/urdf/obj_0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 scale=1 1 1

File: agimus_demo_07_tiago_pro_pick_and_drop/urdf/obj_20.urdf (robot description, URDF)
Before this commit: robot obj_000020, 1 links, 0 joints
Links:
- link base_link: geometry collision mesh filename=package://agimus_demo_07_tiago_pro_pick_and_drop/urdf/obj_2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 scale=1 1 1; visual mesh filename=package://agimus_demo_07_tiago_pro_pick_and_drop/urdf/obj_2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 scale=1 1 1

File: agimus_demo_07_tiago_pro_pick_and_drop/urdf/obj_21.urdf (robot description, URDF)
Before this commit: robot obj_000021, 1 links, 0 joints
Links:
- link base_link: geometry collision mesh filename=package://agimus_demo_07_tiago_pro_pick_and_drop/urdf/obj_2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 scale=1 1 1; visual mesh filename=package://agimus_demo_07_tiago_pro_pick_and_drop/urdf/obj_2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 scale=1 1 1

File: agimus_demo_07_tiago_pro_pick_and_drop/urdf/obj_25.urdf (robot description, URDF)
Before this commit: robot obj_000025, 1 links, 0 joints
Links:
- link base_link: geometry collision mesh filename=package://agimus_demo_07_tiago_pro_pick_and_drop/urdf/obj_2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 scale=1 1 1; visual mesh filename=package://agimus_demo_07_tiago_pro_pick_and_drop/urdf/obj_2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 scale=1 1 1

File: agimus_demo_07_tiago_pro_pick_and_drop/urdf/obj_26.urdf (robot description, URDF)
Before this commit: robot obj_000026, 1 links, 0 joints
Links:
- link base_link: geometry collision mesh filename=package://agimus_demo_07_tiago_pro_pick_and_drop/urdf/obj_2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 scale=1 1 1; visual mesh filename=package://agimus_demo_07_tiago_pro_pick_and_drop/urdf/obj_2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 scale=1 1 1
