Commit message: Adapt box size

File: agimus_demo_07_tiago_pro_pick_and_drop/urdf/box.urdf (robot description, URDF)
Before this commit: robot box, 6 links, 5 joints
Links:
- link box_bottom_link: geometry collision box size=0.295 0.195 0.003; visual box size=0.295 0.195 0.003
- link box_wall_back_link: geometry collision box size=0.003 0.195 0.142; visual box size=0.003 0.195 0.142
- link box_wall_front_link: geometry collision box size=0.003 0.195 0.142; visual box size=0.003 0.195 0.142
- link box_wall_left_link: geometry collision box size=0.295 0.003 0.142; visual box size=0.295 0.003 0.142
- link box_wall_right_link: geometry collision box size=0.295 0.003 0.142; visual box size=0.295 0.003 0.142
Joints:
- joint box_wall_back_joint: origin xyz=-0.0765 0 0.043 rpy=0 0 0 -> xyz=-0.146 0 0.074 rpy=0 0 0
- joint box_wall_front_joint: origin xyz=0.0765 0 0.043 rpy=0 0 0 -> xyz=0.146 0 0.074 rpy=0 0 0
- joint box_wall_left_joint: origin xyz=0 0.0765 0.043 rpy=0 0 0 -> xyz=0 0.096 0.074 rpy=0 0 0
- joint box_wall_right_joint: origin xyz=0 -0.0765 0.043 rpy=0 0 0 -> xyz=0 -0.096 0.074 rpy=0 0 0
