Commit message: Change navigation goals + adapt params + adapt object

File: agimus_demo_07_tiago_pro_pick_and_drop/urdf/obj_22.urdf (robot description, URDF)
Before this commit: robot obj_000022, 1 links, 0 joints
Links:
- link base_link: geometry collision mesh filename=package://agimus_demo_07_tiago_pro_pick_and_drop/urdf/obj_2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; visual mesh filename=package://agimus_demo_07_tiago_pro_pick_and_drop/urdf/obj_2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
